Commit message: Initial commit of Target system package

File: urdf/integeration.xacro (robot description, xacro)
@@ -6,4 +6,5 @@
   <xacro:include filename="treatement_equip.xacro"/>
   <!-- Define the position of the equip with respect to the camera -->
-  <xacro:kinect xyz="0 0 -0.05" rpy="0 3.141592653589793 3.141592653589793" parent_frame="base_link" />
+  <xacro:kinect xyz="0.08 0.09 -0.18" rpy="0 3.141592653589793 -1.57079632679" parent_frame="base_link" />
+  <!-- <xacro:kinect xyz="0.15 0.09 -0.18" rpy="0 3.53429 -1.57079632679" parent_frame="base_link" /> -->
 </robot>

File: urdf/kinect.xacro (robot description, xacro)
@@ -25,5 +25,5 @@
     <inertial>
       <mass value="0.01" />
-      <origin xyz="0 0 0" />
+      <origin xyz="0 0 0"/>
       <inertia ixx="0.001" ixy="0.0" ixz="0.0"
         iyy="0.001" iyz="0.0"
@@ -31,5 +31,5 @@
     </inertial>
     <visual>
-      <origin xyz=" 0 0 0 " rpy="0 0 0" />
+      <origin xyz=" 0 0 0 " rpy="0 0 1.5707963267948966" />
       <geometry>
         <mesh filename="package://treatement_cv/meshes/kinect.dae"/>
@@ -44,5 +44,5 @@
   </link>
   <joint name="camera_depth_joint" type="fixed">
-    <origin xyz="0 0.011 0" rpy="0 0 -1.5707963267949" />
+    <origin xyz="0 0.011 0" rrpy="0 0 0"/>
     <parent link="camera_link" />
     <child link="camera_depth_frame" />
@@ -51,5 +51,5 @@
     <inertial>
       <mass value="0.01" />
-      <origin xyz="0 0 0" />
+      <origin xyz="0 0 0"/>
       <inertia ixx="0.001" ixy="0.0" ixz="0.0"
         iyy="0.001" iyz="0.0"
@@ -65,5 +65,5 @@
     <inertial>
       <mass value="0.001" />
-      <origin xyz="0 0 0" />
+      <origin xyz="0 0 0"/>
       <inertia ixx="0.0001" ixy="0.0" ixz="0.0"
         iyy="0.0001" iyz="0.0"
@@ -72,5 +72,5 @@
   </link>
   <joint name="camera_rgb_joint" type="fixed">
-    <origin xyz="0 -0.012 0" rpy="0 0 -1.5707963267949" />
+    <origin xyz="0 -0.012 0" rpy="0 0 0" />
     <parent link="camera_link" />
     <child link="camera_rgb_frame" />
@@ -79,5 +79,5 @@
     <inertial>
       <mass value="0.001" />
-      <origin xyz="0 0 0" />
+      <origin xyz="0 0 0"/>
       <inertia ixx="0.0001" ixy="0.0" ixz="0.0"
         iyy="0.0001" iyz="0.0"
@@ -93,5 +93,5 @@
     <inertial>
       <mass value="0.001" />
-      <origin xyz="0 0 0" />
+      <origin xyz="0 0 0"/>
       <inertia ixx="0.0001" ixy="0.0" ixz="0.0"
         iyy="0.0001" iyz="0.0"

File: urdf/my_integ.urdf (robot description, URDF)
Before this commit: robot my_integ, 10 links, 9 joints
Joints:
- joint base_camera_joint: origin xyz=0 0 -0.05 rpy=0 3.141592653589793 3.141592653589793 -> xyz=0.08 0.09 -0.18 rpy=0 3.141592653589793 -1.57079632679
- joint base_footprint_to_base_joint: origin xyz=0 0 0.25 rpy=0 3.141592653589793 0 -> xyz=0.0 0.0 0.93 rpy=0 3.141592653589793 3.141592653589793
- joint camera_depth_joint: origin xyz=0 0.011 0 rpy=0 0 -1.5707963267949 -> xyz=0 0.011 0
- joint camera_rgb_joint: origin xyz=0 -0.012 0 rpy=0 0 -1.5707963267949 -> xyz=0 -0.012 0 rpy=0 0 0

File: urdf/treatement_equip.xacro (robot description, xacro)
@@ -43,6 +43,6 @@
   <joint name="base_footprint_to_base_joint" type="fixed">
     <origin
-      xyz="0 0 0.25"
-      rpy="0 3.141592653589793 0" />
+      xyz="0.0 0.0 0.93"
+      rpy="0 3.141592653589793 3.141592653589793" />
     <parent
       link="base_footprint" />
